File: Hardware/Basic/Top/Smartwatch-BASIC-TOP.sch (EAGLE design)
At the start: 59 parts, among them SW6 SWITCH.MOM, SW7 SWITCH.MOM, U2 NRF52832_MODULE_MDBT42, U4 FT231XS

Commit message: Header Pins Fixed
Parts:
- J1: device LinnesLab-Connectors:CONN_07 -> LinnesLab-Connectors:CONN_07-1.27MM
Changed lines of the file:
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@@
 <part name="SW6" library="LinnesLab-Switches" deviceset="SWITCH.MOM" device=""/>
 <part name="SW7" library="LinnesLab-Switches" deviceset="SWITCH.MOM" device=""/>
-<part name="J1" library="LinnesLab-Connectors" deviceset="CONN_07" device=""/>
+<part name="J1" library="LinnesLab-Connectors" deviceset="CONN_07" device="-1.27MM"/>
 <part name="R10" library="LinnesLab-Passives" deviceset="RESISTOR" device="0603" package3d_urn="urn:adsk.eagle:package:15661944/2" value="27"/>
 <part name="R16" library="LinnesLab-Passives" deviceset="RESISTOR" device="0603" package3d_urn="urn:adsk.eagle:package:15661944/2" value="27"/>

Commit message: Top Board airwire fixed
Parts:
- removed LED5: RED, LinnesLab-LED:LED0603
- removed LED6: YELLOW, LinnesLab-LED:LED0603
- removed R18: 1k, LinnesLab-Passives:RESISTOR0603
- added LED1: RED, LinnesLab-LED:LED0603
- added LED2: BLUE, LinnesLab-LED:LED0603
- added R9: 27, LinnesLab-Passives:RESISTOR0603
- LED4: value BLUE -> YELLOW
- R10: value 27 -> 4.7k
- R11: value (none) -> 100k
- R14: value 100k -> 27
- R16: value 27 -> 1k
- renumbered D4 to D2, D5 to D3, L2 to L1, R17 to R15, SW6 to SW2, SW7 to SW1
Connections:
- net 3.3V: now also LED3.A, LED4.A; no longer LED5.A, LED6.A
- net A4/BATT: now also R12.1, R13.2; no longer R13.1, R14.2
- net D27/CHRG.STAT: now also R11.1; no longer R12.1
- net GND: now also LED1.C, LED2.C, R10.1, R13.1; no longer LED3.C, LED4.C, R11.1, R14.1
- net N$10: now also LED2.A; no longer LED4.A
- net N$16: now also R10.2; no longer R11.2
- net N$25: now also R9.2; no longer R10.2
- net N$26: now also R14.2; no longer R16.2
- net N$27: now also LED3.C; no longer LED5.C
- net N$28: now also LED4.C, R16.2; no longer LED6.C, R18.2
- net N$9: now also LED1.A; no longer LED3.A
- net TXLED: now also R16.1; no longer R18.1
- net USB+: now also R14.1; no longer R16.1
- net USB-: now also R9.1; no longer R10.1
- net VIN: now also R11.2; no longer R12.2
- net VLIPO: now also R12.2; no longer R13.2
Other:
- moved on the sheet: LED3, LED4, R10, R11, R12, R13, R14, R16

Commit message: Top Board BOM WIP
Parts:
- removed C22, C23: 47p, LinnesLab-Passives:CAPACITOR0603
- removed U4: FT231XS, LinnesLab-DigitalIC:FT231XS
- added C2: 10u, LinnesLab-Passives:CAPACITOR0805
- added C20: 4.7u, LinnesLab-Passives:CAPACITOR0603
- added U1: NRF52832_MODULE_MDBT42, LinnesLab-Microcontrollers:NRF52832_MODULE_MDBT42
- C1: value 4.7u -> 1u
- C10, C11: value 300p -> 2.2uF; device LinnesLab-Passives:CAPACITOR0603 -> LinnesLab-Passives:CAPACITOR0402
- C12: value 10u -> 2.2uF; device LinnesLab-Passives:CAPACITOR0805 -> LinnesLab-Passives:CAPACITOR0402
- C13, C18: value 2.2uF -> 100n; device LinnesLab-Passives:CAPACITOR0402 -> LinnesLab-Passives:CAPACITOR0603
- C14: value 100n -> 4.7u
- C15, C17: value 2.2uF -> 47p; device LinnesLab-Passives:CAPACITOR0402 -> LinnesLab-Passives:CAPACITOR0603
- C16: value 10uF -> 1u
- C19: value 2.2uF -> 1u; device LinnesLab-Passives:CAPACITOR0402 -> LinnesLab-Passives:CAPACITOR0603
- C3: value 4.7u -> (none)
- C4: value 100n -> (none)
- C5, C6: value 1u -> 300p
- C7: value 1u -> 10uF
- C8, C9: value (none) -> 2.2uF; device LinnesLab-Passives:CAPACITOR0603 -> LinnesLab-Passives:CAPACITOR0402
- R10: value 4.7k -> 27
- R11: value 100k -> 4.7k
- R14: value 27 -> 100k
- R6: value 10k -> 390k
- R7: value 390k -> 10k
- SW1: value SWITCH.MOM -> (none); device LinnesLab-Switches:SWITCH.MOM -> LinnesLab-Switches:SPST-PTS830GG140-COPY.1-3
- SW3: value (none) -> SWITCH.MOM; device LinnesLab-Switches:SPST-PTS830GG140-COPY.1-3 -> LinnesLab-Switches:SWITCH.MOM
- U2: value NRF52832_MODULE_MDBT42 -> (none); device LinnesLab-Microcontrollers:NRF52832_MODULE_MDBT42 -> LinnesLab-Displays:DISP_OLED_UG-2864HSWEG01-NO-WRAPAROUND
- U3: value (none) -> FT231XS; device LinnesLab-Displays:DISP_OLED_UG-2864HSWEG01-NO-WRAPAROUND -> LinnesLab-DigitalIC:FT231XS
- renumbered CHRG2 to CHRG1, CORTEX1 to DEBUG1, JP2 to JP1, LDO2 to LDO1, USB2 to USB1, XTAL2 to XTAL1
Connections:
- removed net N$21 (its old number): SW1.3, SW1.4
- new net N$22: SW3.3, SW3.4
- net !CTS: now also U3.!CTS; no longer U4.!CTS
- net !DTR: now also U3.!DTR; no longer U4.!DTR
- net 3.3V: now also C11.2, C18.2, C19.1, C2.2, R12.2, R7.2, U1.VDD, U2.VBAT, U3.!RESET, U3.VCCIO; no longer C17.2, C19.2, C4.2, C6.1, R5.2, R8.2, U3.VBAT, U3.VDD, U4.!RESET, U4.VCCIO
- net A4/BATT: now also R13.1, R14.2, U1.P0.28/AIN4; no longer R12.1, R13.2, U2.P0.28/AIN4
- net A6/TIA: now also U1.P0.30/AIN6; no longer U2.P0.30/AIN6
- net A7/PPG: now also U1.P0.31/AIN7; no longer U2.P0.31/AIN7
- net D11/SW1: now also SW2.1, U1.P0.11; no longer SW1.1, U2.P0.11
- net D15/SW2: now also SW3.1, U1.P0.15; no longer SW2.1, U2.P0.15
- net D16/CS.OLED: now also U1.P0.16, U2./CS; no longer U2.P0.16, U3./CS
- net D27/CHRG.STAT: now also R8.1, U1.P0.27; no longer R11.1, U2.P0.27
- net D29/LED.CTRL: now also U1.P0.29/AIN5; no longer U2.P0.29/AIN5
- net D3/RESET.OLED: now also U1.P0.03/AIN1, U2./RES; no longer U2.P0.03/AIN1, U3./RES
- net D4/DC.OLED: now also U1.P0.04/AIN2, U2.DC/I2C_SA0; no longer U2.P0.04/AIN2, U3.DC/I2C_SA0
- net D5/CD1: now also U1.P0.05/AIN3; no longer U2.P0.05/AIN3
- net D7/SD.CS: now also U1.P0.07; no longer U2.P0.07
- net DFU: now also SW1.B, U1.P0.20; no longer SW3.B, U2.P0.20
- net DTR: now also C13.1; no longer C14.1
- net FRST: now also U1.P0.22; no longer U2.P0.22
- net FT3V3: now also U3.3V3OUT; no longer U4.3V3OUT
- net GND: now also C1.2, C11.1, C14.1, C15.1, C17.2, C19.2, C2.1, C20.2, C3.1, C4.2, C5.2, C7.1, C9.1, R11.1, R12.1, R14.1, R5.1, R6.2, SW1.A, U1.GND@1, U1.GND@2, U1.GND@3, U1.GND@4, U2.BS0, U2.BS2, U2.NC(GND)@1, U2.NC(GND)@2, U2.VLSS, U2.VSS, U3.GND@16, U3.GND@6; no longer C1.1, C10.2, C11.2, C17.1, C19.1, C22.2, C23.1, C3.2, C4.1, C5.1, C7.2, C8.1, C9.2, R10.1, R13.1, R6.1, R7.2, R8.1, SW3.A, U2.GND@1, U2.GND@2, U2.GND@3, U2.GND@4, U3.BS0, U3.BS2, U3.NC(GND)@1, U3.NC(GND)@2, U3.VLSS, U3.VSS, U4.GND@16, U4.GND@6
- net LED1: now also U1.P0.17; no longer U2.P0.17
- net LED2: now also U1.P0.19; no longer U2.P0.19
- net MISO: now also U1.P0.14; no longer U2.P0.14
- net MOSI: now also U1.P0.13, U2.D1/SPI_SDIN/I2C_SDA; no longer U2.P0.13, U3.D1/SPI_SDIN/I2C_SDA
- net N$1: now also R5.2, U2.BS1; no longer R6.2, U3.BS1
- net N$11: now also U1.DCC; no longer U2.DCC
- net N$12: now also C1.1, U1.DEC4; no longer C7.1, U2.DEC4
- net N$13: now also C7.2, U2.VCC; no longer C16.2, U3.VCC
- net N$15: now also C9.2, U2.VCOMH; no longer C18.2, U3.VCOMH
- net N$16: now also R11.2; no longer R10.2
- net N$2: now also R6.1, U2.IREF; no longer R7.1, U3.IREF
- net N$25: now also U3.USBDM; no longer U4.USBDM
- net N$26: now also R10.2, U3.USBDP; no longer R14.2, U4.USBDP
- net N$3: now also C10.2, U2.C2P; no longer C13.2, U3.C2P
- net N$4: now also C3.2, U1.P0.00/XL1; no longer C8.2, U2.P0.00/XL1
- net N$5: now also C10.1, U2.C2N; no longer C13.1, U3.C2N
- net N$6: now also C4.1, U1.P0.01/XL2; no longer C9.1, U2.P0.01/XL2
- net N$7: now also C8.2, U2.C1P; no longer C15.2, U3.C1P
- net N$8: now also C8.1, U2.C1N; no longer C15.1, U3.C1N
- net P0.09/NFC1: now also C5.1, U1.P0.09; no longer C11.1, U2.P0.09
- net P0.10/NFC2: now also C6.1, U1.P0.10; no longer C10.1, U2.P0.10
- net RESET: now also C13.2, R7.1, U1.P0.21/RESET; no longer C14.2, R5.1, U2.P0.21/RESET
- net RXD: now also U1.P0.08, U3.RXD; no longer U2.P0.08, U4.RXD
- net RXLED: now also U3.CBUS1; no longer U4.CBUS1
- net SCK: now also U1.P0.12, U2.D0/SPI_SCLK/I2C_SCK; no longer U2.P0.12, U3.D0/SPI_SCLK/I2C_SCK
- net SCL: now also U1.P0.26; no longer U2.P0.26
- net SDA: now also U1.P0.25; no longer U2.P0.25
- net SWCLK: now also U1.SWDCLK; no longer U2.SWDCLK
- net SWDIO: now also U1.SWDIO; no longer U2.SWDIO
- net SWO: now also U1.P0.18/SWO; no longer U2.P0.18/SWO
- net TXD: now also U1.P0.06, U3.TXD; no longer U2.P0.06, U4.TXD
- net TXLED: now also U3.CBUS2; no longer U4.CBUS2
- net USB+: now also C17.1, R10.1; no longer C22.1, R14.1
- net USB-: now also C15.2; no longer C23.2
- net VIN: now also C14.2, C16.2, R8.2; no longer C1.2, C5.2, R11.2
- net VLIPO: now also C20.1, R13.2; no longer C3.1, R12.2
- net V_USB: now also U3.VCC; no longer U4.VCC
Other:
- moved on the sheet: C1, C10, C11, C12, C13, C14, C15, C16, C17, C18, C19, C3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
